File: kicad/amplifier/amboulons/amboulons.sch (KiCad schematic (older format))
At the start: 36 parts, among them J1 Screw_Terminal_01x02, J2 Screw_Terminal_01x02, J3 Screw_Terminal_01x02, J4 Screw_Terminal_01x03, J5 Screw_Terminal_01x02, Q1 BC549, Q2 BC549, U1 EL84, U2 ECC83, U3 EL84

Commit message: update for version 1.1
Parts:
- added TP1, TP2: TestPoint_Probe, TestPoint:TestPoint_THTPad_D1.0mm_Drill0.5mm, symbol Connector:TestPoint_Probe
Connections:
- net at R3.1, U1.3 (K_G3): now also TP1.1
- net at R11.1, U3.3 (K_G3): now also TP2.1
Changed lines of the file:
@@
 $EndComp
 Wire Wire Line
-	2200 2400 2200 2250
-Wire Wire Line
-	4700 2400 4700 2250
+	2200 2400 2200 2300
+Wire Wire Line
+	4700 2400 4700 2300
 Wire Wire Line
 	4700 2700 4700 2900
@@
 Wire Wire Line
 	2200 4900 2350 4900
+$Comp
+L Connector:TestPoint_Probe TP2
+U 1 1 5F11EDCA
+P 4850 2300
+F 0 "TP2" H 5003 2401 50  0000 L CNN
+F 1 "TestPoint_Probe" H 5003 2310 50  0000 L CNN
+F 2 "TestPoint:TestPoint_THTPad_D1.0mm_Drill0.5mm" H 5050 2300 50  0001 C CNN
+F 3 "~" H 5050 2300 50  0001 C CNN
+	1    4850 2300
+	1    0    0    -1
+$EndComp
+Wire Wire Line
+	4850 2300 4700 2300
+Connection ~ 4700 2300
+Wire Wire Line
+	4700 2300 4700 2250
+$Comp
+L Connector:TestPoint_Probe TP1
+U 1 1 5F123D95
+P 2050 2300
+F 0 "TP1" V 2340 2355 50  0000 C CNN
+F 1 "TestPoint_Probe" V 2249 2355 50  0000 C CNN
+F 2 "TestPoint:TestPoint_THTPad_D1.0mm_Drill0.5mm" H 2250 2300 50  0001 C CNN
+F 3 "~" H 2250 2300 50  0001 C CNN
+	1    2050 2300
+	0    -1   -1   0
+$EndComp
+Wire Wire Line
+	2050 2300 2200 2300
+Connection ~ 2200 2300
+Wire Wire Line
+	2200 2300 2200 2250
 $EndSCHEMATC
